File: KiCad/tn9k_f18a_compact/tn9k_f18a.kicad_pcb (KiCad board)
At the start: 2 copper layers, 32 x 94.9 mm, 27 parts, among them J2 VGA, J3 Tang Nano 9k, J4 TN9k/2, J5 VGA, J6 VGA, U1 1G08, U4 74LCX16245

Commit message: Version H1 sent to aisler
Other:
- board text added: "TANG NANO 9K F18A - Version H1 2023 Luis Antoniosi, Hans Hübner https://github.com/lfantoniosi/tn9k_f18a"
- board text removed: "TANG NANO 9K F18A 2023 Luis Antoniosi, Hans Hübner https://github.com/lfantoniosi/tn9k_f18a"
Changed lines of the file:
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@@
   (gr_line (start 128.778 128.143) (end 126.492 128.143)
     (stroke (width 0.1) (type default)) (layer "Edge.Cuts"))
-  (gr_text "TANG NANO 9K F18A\n2023 Luis Antoniosi, Hans Hübner\nhttps://github.com/lfantoniosi/tn9k_f18a" (at 118.618 67.945 90) (layer "B.SilkS")
+  (gr_text "TANG NANO 9K F18A - Version H1\n2023 Luis Antoniosi, Hans Hübner\nhttps://github.com/lfantoniosi/tn9k_f18a" (at 118.618 67.945 90) (layer "B.SilkS")
     (effects (font (size 1.5 1.5) (thickness 0.25) bold) (justify left bottom mirror))
   )
