File: KiCad/tn_vdp_v1_compact/tn_vdp_v1_compact.kicad_pcb (KiCad board)
At the start: 2 copper layers, 32 x 94.9 mm, 28 parts, among them J2 VGA, J3 Tang Nano 9k, J4 TN9k/2, J5 VGA, J6 VGA, U1 1G08, U4 74LCX16245

Commit message: rebrand of the compact version + license update
Other:
- board text added: "tn_vdp_v1_compact - Version H2 2023 Luis Antoniosi, Hans Hübner https://github.com/lfantoniosi/tn_vdp"
- board text removed: "TANG NANO 9K F18A - Version H1 2023 Luis Antoniosi, Hans Hübner https://github.com/lfantoniosi/tn9k_f18a"
