File: kicad/tn_vdp_v3_board/tn_vdp_v3_board.kicad_pcb (KiCad board)
At the start: 2 copper layers, 49.4 x 67.8 mm, 18 parts, among them J1 Conn_02x10_Odd_Even, J2 Conn_02x10_Odd_Even, J3 Conn_01x20, J4 Conn_02x04_Counter_Clockwise, J6 Conn_01x20, U1 SN74LVC245, U2 SN74LVC245, U3 SN74LVC245, U4 MCP3202

Commit message: improving stability and precision of clock dividers
Parts:
- added C5: C_Polarized_US, Capacitor_THT:CP_Radial_D5.0mm_P2.50mm, F.Cu at (168.8, 109.4)
- added C6: 102, Capacitor_THT:C_Disc_D5.0mm_W2.5mm_P2.50mm, F.Cu at (170.4, 102.0)
- added J5: Conn_01x02, Connector_PinHeader_2.54mm:PinHeader_1x02_P2.54mm_Horizontal, F.Cu at (150.3, 102.6)
Connections:
- J1 pad 8: AUDIO -> unconnected-(J1-Pin_8-Pad8)
- J2 pad 8: AUDIO -> unconnected-(J2-Pin_8-Pad8)
- RV1 pad 2: VREF -> AUDIO_REF
- U4 pad 2: AUDIO -> AUDIO_REF
- U4 pad 3: AUDIO -> AUDIO_REF
- U4 pad 8: VREF -> VCC
Routing:
- net AUDIO: track 116.6 -> 21.3 mm
- net CD1: track 99.6 -> 177.5 mm
- net CD4: track 166.8 -> 104.4 mm, vias 0 -> 1
- net GROMCLK: track 81.5 -> 134.6 mm, vias 0 -> 1
- net USR2_1V8: track 68.1 -> 28.8 mm, vias 2 -> 0
- net ~{CSW}: track 95.7 -> 126.4 mm, vias 3 -> 0
- net CD3_3V3: track 71.3 -> 42.4 mm
- net AUDIO_REF: track 0.00 -> 28.4 mm
- net CD2: track 113.4 -> 87.4 mm, vias 0 -> 2
- net CD0: track 95.2 -> 109.6 mm
- net MODE1_3V3: track 28.3 -> 38.9 mm, vias 2 -> 1
- net VREF: track 20.7 -> 13.1 mm
- net VCC: track 121.5 -> 128.7 mm
- net USR3_1V8: track 38.9 -> 32.0 mm
- net CD5: track 92.0 -> 98.6 mm
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Other:
- board text added: "TN-VDP 20K v1.1 - 2023 RENDERENG - LUIS ANTONIOSI"
- board text removed: "TN-VDP 20K v1.0 - 2023 RENDERENG - LUIS ANTONIOSI"

Commit message: new clocks 3.58Mhz !!!
Parts:
- C5: value C_Polarized_US -> 10uF
Changed lines of the file:
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@@
+        (effects (font (size 1 1) (thickness 0.15)))
+    )
+    (fp_text user "${VALUE}" (at 1.175 2.325 90) (layer "F.SilkS")
         (effects (font (size 1 1) (thickness 0.15)))
     )
@@
         (effects (font (size 1 1) (thickness 0.15)))
     )
-    (fp_text value "C_Polarized_US" (at 1.25 3.75) (layer "F.Fab")
-        (effects (font (size 1 1) (thickness 0.15)))
-    )
-    (fp_text user "102" (at -1.694888 2.5) (layer "F.SilkS")
+    (fp_text value "10uF" (at 1.25 3.75) (layer "F.Fab")
+        (effects (font (size 1 1) (thickness 0.15)))
+    )
+    (fp_text user "${VALUE}" (at -2.3199 -0.025 90) (layer "F.SilkS")
         (effects (font (size 0.8 0.8) (thickness 0.15)))
     )

Commit message: V9958 Socket + New V3 Board (audio fix + cinch connector)
Parts:
- removed H1, H2, H3, H4: MountingHole, MountingHole:MountingHole_2.2mm_M2_ISO7380_Pad
- removed J1: Conn_02x10_Odd_Even, Connector_PinHeader_2.54mm:PinHeader_2x10_P2.54mm_Vertical
- added J7: AUDIO, Connector_BarrelJack:BarrelJack_CUI_PJ-063AH_Horizontal_CircularHoles, F.Cu at (138.5, 105.5)
- moved J5 9.72 mm to (145.0, 94.5), turned to 180 degrees
- moved J2 2.58 mm to (181.8, 71.2)
- moved J3 1.94 mm to (150.0, 48.1)
- moved J6 1.94 mm to (170.3, 48.1)
- moved J4 1.25 mm to (174.7, 77.2)
- moved C6 1.05 mm to (170.4, 101.0)
- moved C5 0.90 mm to (168.8, 108.5)
Connections:
- C4 pad 1: VREF -> VCC
Routing:
- net CD1: track 177.5 -> 68.9 mm, vias 2 -> 1
- net GROMCLK: track 134.6 -> 49.0 mm, vias 1 -> 0
- net ~{CSW}: track 126.4 -> 57.2 mm, vias 0 -> 1
- net ~{RESET}: track 113.8 -> 56.1 mm, vias 0 -> 1
- net ~{INT}: track 92.1 -> 37.5 mm
- net CD0: track 109.6 -> 67.7 mm
- net MODE: track 111.2 -> 70.7 mm, vias 1 -> 0
- net MODE1_3V3: track 38.9 -> 66.1 mm, vias 1 -> 0
- net MODE1: track 92.4 -> 67.3 mm, vias 0 -> 1
- net AUDIO: track 21.3 -> 44.6 mm
- net CD2: track 87.4 -> 66.0 mm, vias 2 -> 1
- net VCC: track 128.7 -> 109.2 mm
- net CD4: track 104.4 -> 85.7 mm
- net CPUCLK: track 66.5 -> 49.5 mm, vias 1 -> 2
- net CD5: track 98.6 -> 82.2 mm
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Other:
- board text added: "TN-VDP 20K v2.01 - 2023 RENDERENG - LUIS ANTONIOSI"
- board text removed: "TN-VDP 20K v1.1 - 2023 RENDERENG - LUIS ANTONIOSI"

Commit message: v3 last board  last version
Parts:
- J7: value AUDIO -> Barrel_Jack_MountingPin
- moved J7 0.69 mm to (137.9, 105.8)
Connections:
- J7 pad 1: AUDIO -> GND
- J7 pad 2: GND -> AUDIO
- J7 pad MP: (no net) -> GND
Routing:
- net CD0: track 67.7 -> 152.3 mm, vias 2 -> 0
- net CD5: track 82.2 -> 146.2 mm, vias 1 -> 0
- net ~{CSR}: track 138.8 -> 95.1 mm
- net CD2: track 66.0 -> 97.0 mm
- net MODE1_3V3: track 66.1 -> 36.9 mm
- net USR4_1V8: track 53.3 -> 27.9 mm
- net CD1: track 68.9 -> 89.2 mm, vias 1 -> 0
- net CD7: track 93.0 -> 82.2 mm
- net CD4: track 85.7 -> 95.9 mm, vias 1 -> 2
- net MODE1: track 67.3 -> 76.8 mm, vias 1 -> 0
- net ~{CSW}: track 57.2 -> 66.7 mm, vias 1 -> 2
- net ~{RESET}: track 56.1 -> 48.8 mm, vias 1 -> 0
- net CD6: track 95.7 -> 89.1 mm, vias 1 -> 0
- net ~{INT}: track 37.5 -> 44.0 mm, vias 0 -> 1
- net AUDIO: track 44.6 -> 39.5 mm
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Other:
- board text added: "TN-VDP 20K v2.02 - 2023 RENDERENG - LUIS ANTONIOSI"
- board text removed: "TN-VDP 20K v2.01 - 2023 RENDERENG - LUIS ANTONIOSI"
