File: kicad/tn_vdp_v3_board/tn_vdp_v3_board.kicad_sch (KiCad schematic)
At the start: 18 parts, among them J1 Conn_02x10_Odd_Even, J2 Conn_02x10_Odd_Even, J3 Conn_01x20, J4 Conn_02x04_Counter_Clockwise, J6 Conn_01x20, U1 SN74LVC245, U2 SN74LVC245, U3 SN74LVC245, U4 MCP3202

Commit message: improving stability and precision of clock dividers
Parts:
- added C5: C_Polarized_US, Capacitor_THT:CP_Radial_D5.0mm_P2.50mm, symbol Device:C_Polarized_US
- added C6: 102, Capacitor_THT:C_Disc_D5.0mm_W2.5mm_P2.50mm, symbol Device:C
- added J5: Conn_01x02, Connector_PinHeader_2.54mm:PinHeader_1x02_P2.54mm_Horizontal, symbol Connector_Generic:Conn_01x02
Connections:
- net AUDIO: now also C5.1, J5.1 (Pin_1); no longer J1.8 (Pin_8), J2.8 (Pin_8), U4.2 (CH0), U4.3 (CH1)
- net GND: now also C6.2, J5.2 (Pin_2)
- net VCC: now also U4.8 (VDD/VREF)
- net VREF: no longer RV1.2, U4.8 (VDD/VREF)
- new net AUDIO_REF: C5.2, C6.1, RV1.2, U4.2 (CH0), U4.3 (CH1)
- no-connect marks 2 -> 4
Changed lines of the file:
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@@
 (kicad_sch (version 20230121) (generator eeschema)
   (paper "A4")
+  (junction (at 93.98 111.76) (diameter 0) (color 0 0 0 0)
+  )
+  (no_connect (at 82.55 29.21))
   (no_connect (at 226.06 20.32))
+  (no_connect (at 43.18 30.48))
   (no_connect (at 49.53 -41.91))
+  (wire (pts (xy 93.98 111.76) (xy 93.98 114.3))
+    (stroke (width 0) (type default))
+  )
+  (wire (pts (xy 96.52 111.76) (xy 93.98 111.76))
+    (stroke (width 0) (type default))
+  )
+  (wire (pts (xy 91.44 111.76) (xy 93.98 111.76))
+    (stroke (width 0) (type default))
+  )
   (global_label "GND" (shape input) (at 30.48 22.86 180) (fields_autoplaced)
     (effects (font (size 1.27 1.27)) (justify right))
@@
     )
   )
+  (global_label "AUDIO_REF" (shape input) (at 275.59 72.39 90) (fields_autoplaced)
+    (effects (font (size 1.27 1.27)) (justify left))
+    (property "Intersheetrefs" "${INTERSHEET_REFS}" (at 275.59 59.3846 90)
+      (effects (font (size 1.27 1.27)) (justify left) hide)
+    )
+  )
   (global_label "GND" (shape input) (at 148.59 137.16 270) (fields_autoplaced)
     (effects (font (size 1.27 1.27)) (justify right))
@@
     )
   )
-  (global_label "VREF" (shape input) (at 76.2 68.58 90) (fields_autoplaced)
-    (effects (font (size 1.27 1.27)) (justify left))
-    (property "Intersheetrefs" "${INTERSHEET_REFS}" (at 76.2 61.078 90)
+  (global_label "VCC" (shape input) (at 76.2 68.58 90) (fields_autoplaced)
+    (effects (font (size 1.27 1.27)) (justify left))
+    (property "Intersheetrefs" "${INTERSHEET_REFS}" (at 76.2 62.0456 90)
       (effects (font (size 1.27 1.27)) (justify left) hide)
     )
@@
     )
   )
-  (global_label "AUDIO" (shape input) (at 63.5 76.2 180) (fields_autoplaced)
-    (effects (font (size 1.27 1.27)) (justify right))
-    (property "Intersheetrefs" "${INTERSHEET_REFS}" (at 54.9698 76.2 0)
+  (global_label "AUDIO_REF" (shape input) (at 63.5 76.2 180) (fields_autoplaced)
+    (effects (font (size 1.27 1.27)) (justify right))
+    (property "Intersheetrefs" "${INTERSHEET_REFS}" (at 50.4946 76.2 0)
       (effects (font (size 1.27 1.27)) (justify right) hide)
     )
@@
     )
   )
+  (global_label "GND" (shape input) (at 31.75 55.88 180) (fields_autoplaced)
+    (effects (font (size 1.27 1.27)) (justify right))
+    (property "Intersheetrefs" "${INTERSHEET_REFS}" (at 24.9737 55.88 0)
+      (effects (font (size 1.27 1.27)) (justify right) hide)
+    )
+  )
   (global_label "GROMCLK_3V3" (shape input) (at 201.93 55.88 180) (fields_autoplaced)
     (effects (font (size 1.27 1.27)) (justify right))
@@
     )
   )
-  (global_label "AUDIO" (shape input) (at 63.5 86.36 180) (fields_autoplaced)
-    (effects (font (size 1.27 1.27)) (justify right))
-    (property "Intersheetrefs" "${INTERSHEET_REFS}" (at 54.9698 86.36 0)
+  (global_label "AUDIO_REF" (shape input) (at 63.5 86.36 180) (fields_autoplaced)
+    (effects (font (size 1.27 1.27)) (justify right))
+    (property "Intersheetrefs" "${INTERSHEET_REFS}" (at 50.4946 86.36 0)
       (effects (font (size 1.27 1.27)) (justify right) hide)
     )
@@
     )
   )
+  (global_label "AUDIO_REF" (shape input) (at 93.98 114.3 270) (fields_autoplaced)
+    (effects (font (size 1.27 1.27)) (justify right))
+    (property "Intersheetrefs" "${INTERSHEET_REFS}" (at 93.98 127.3054 90)
+      (effects (font (size 1.27 1.27)) (justify right) hide)
+    )
+  )
   (global_label "GROMCLK" (shape input) (at 43.18 27.94 0) (fields_autoplaced)
     (effects (font (size 1.27 1.27)) (justify left))
@@
     )
   )
-  (global_label "VREF" (shape input) (at 91.44 111.76 0) (fields_autoplaced)
-    (effects (font (size 1.27 1.27)) (justify left))
-    (property "Intersheetrefs" "${INTERSHEET_REFS}" (at 98.942 111.76 0)
+  (global_label "AUDIO" (shape input) (at 104.14 111.76 0) (fields_autoplaced)
+    (effects (font (size 1.27 1.27)) (justify left))
+    (property "Intersheetrefs" "${INTERSHEET_REFS}" (at 112.6702 111.76 0)
       (effects (font (size 1.27 1.27)) (justify left) hide)
     )
@@
     )
   )
+  (global_label "GND" (shape input) (at 275.59 80.01 270) (fields_autoplaced)
+    (effects (font (size 1.27 1.27)) (justify right))
+    (property "Intersheetrefs" "${INTERSHEET_REFS}" (at 275.59 86.7863 90)
+      (effects (font (size 1.27 1.27)) (justify right) hide)
+    )
+  )
   (global_label "CD7" (shape input) (at 69.85 44.45 180) (fields_autoplaced)
     (effects (font (size 1.27 1.27)) (justify right))
@@
     )
   )
+  (global_label "AUDIO" (shape input) (at 31.75 53.34 180) (fields_autoplaced)
+    (effects (font (size 1.27 1.27)) (justify right))
+    (property "Intersheetrefs" "${INTERSHEET_REFS}" (at 23.2198 53.34 0)
+      (effects (font (size 1.27 1.27)) (justify right) hide)
+    )
+  )
   (global_label "USR2_1V8" (shape input) (at 201.93 63.5 180) (fields_autoplaced)
     (effects (font (size 1.27 1.27)) (justify right))
@@
     (property "Intersheetrefs" "${INTERSHEET_REFS}" (at 182.7561 106.68 0)
       (effects (font (size 1.27 1.27)) (justify right) hide)
-    )
-  )
-  (global_label "AUDIO" (shape input) (at 82.55 29.21 0) (fields_autoplaced)
-    (effects (font (size 1.27 1.27)) (justify left))
-    (property "Intersheetrefs" "${INTERSHEET_REFS}" (at 91.0802 29.21 0)
-      (effects (font (size 1.27 1.27)) (justify left) hide)
-    )
-  )
-  (global_label "AUDIO" (shape input) (at 43.18 30.48 0) (fields_autoplaced)
-    (effects (font (size 1.27 1.27)) (justify left))
-    (property "Intersheetrefs" "${INTERSHEET_REFS}" (at 51.7102 30.48 0)
-      (effects (font (size 1.27 1.27)) (justify left) hide)
     )
   )
@@
     )
   )
+  (symbol (lib_id "Device:C_Polarized_US") (at 100.33 111.76 270) (unit 1)
+    (in_bom yes) (on_board yes) (dnp no) (fields_autoplaced)
+    (property "Reference" "C5" (at 100.965 105.41 90)
+      (effects (font (size 1.27 1.27)))
+    )
+    (property "Value" "C_Polarized_US" (at 100.965 107.95 90)
+      (effects (font (size 1.27 1.27)))
+    )
+    (property "Footprint" "Capacitor_THT:CP_Radial_D5.0mm_P2.50mm" (at 100.33 111.76 0)
+      (effects (font (size 1.27 1.27)) hide)
+    )
+    (property "Datasheet" "~" (at 100.33 111.76 0)
+      (effects (font (size 1.27 1.27)) hide)
+    )
+    (pin "1")
+    (pin "2")
+    (instances
+      (project "tn_vdp_v3_board"
+        (path "/e3c6ad0b-efa5-4827-958c-c20bf8519fa1"
+          (reference "C5") (unit 1)
+        )
+      )
+    )
+  )
+  (symbol (lib_id "Device:C") (at 275.59 76.2 0) (unit 1)
+    (in_bom yes) (on_board yes) (dnp no) (fields_autoplaced)
+    (property "Reference" "C6" (at 279.4 75.565 0)
+      (effects (font (size 1.27 1.27)) (justify left))
+    )
+    (property "Value" "102" (at 279.4 78.105 0)
+      (effects (font (size 1.27 1.27)) (justify left))
+    )
+    (property "Footprint" "Capacitor_THT:C_Disc_D5.0mm_W2.5mm_P2.50mm" (at 276.5552 80.01 0)
+      (effects (font (size 1.27 1.27)) hide)
+    )
+    (property "Datasheet" "~" (at 275.59 76.2 0)
+      (effects (font (size 1.27 1.27)) hide)
+    )
+    (pin "1")
+    (pin "2")
+    (instances
+      (project "tn_vdp_v3_board"
+        (path "/e3c6ad0b-efa5-4827-958c-c20bf8519fa1"
+          (reference "C6") (unit 1)
+        )
+      )
+    )
+  )
   (symbol (lib_id "tms9118a_sym:SN74LVC245") (at 148.59 50.8 0) (unit 1)
     (in_bom yes) (on_board yes) (dnp no) (fields_autoplaced)
@@
         )
       )
+    )
+  )
+  (symbol (lib_id "Connector_Generic:Conn_01x02") (at 36.83 53.34 0) (unit 1)
+    (in_bom yes) (on_board yes) (dnp no) (fields_autoplaced)
+    (property "Reference" "J5" (at 39.37 53.975 0)
+      (effects (font (size 1.27 1.27)) (justify left))
+    )
+    (property "Value" "Conn_01x02" (at 39.37 56.515 0)
+      (effects (font (size 1.27 1.27)) (justify left))
+    )
+    (property "Footprint" "Connector_PinHeader_2.54mm:PinHeader_1x02_P2.54mm_Horizontal" (at 36.83 53.34 0)
+      (effects (font (size 1.27 1.27)) hide)
+    )
+    (property "Datasheet" "~" (at 36.83 53.34 0)
+      (effects (font (size 1.27 1.27)) hide)
+    )
+    (pin "1")
+    (pin "2")
+    (instances
+      (project "tn_vdp_v3_board"
+        (path "/e3c6ad0b-efa5-4827-958c-c20bf8519fa1"
+          (reference "J5") (unit 1)
+        )
+      )

Commit message: new clocks 3.58Mhz !!!
Parts:
- C5: value C_Polarized_US -> 10uF
Changed lines of the file:
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@@
       (effects (font (size 1.27 1.27)))
     )
-    (property "Value" "C_Polarized_US" (at 100.965 107.95 90)
+    (property "Value" "10uF" (at 100.965 107.95 90)
       (effects (font (size 1.27 1.27)))
     )

Commit message: V9958 Socket + New V3 Board (audio fix + cinch connector)
Parts:
- removed H1, H2, H3, H4: MountingHole, MountingHole:MountingHole_2.2mm_M2_ISO7380_Pad, symbol Mechanical:MountingHole
- removed J1: Conn_02x10_Odd_Even, Connector_PinHeader_2.54mm:PinHeader_2x10_P2.54mm_Vertical, symbol Connector_Generic:Conn_02x10_Odd_Even
- added J7: AUDIO, Connector_BarrelJack:BarrelJack_CUI_PJ-063AH_Horizontal_CircularHoles, symbol Connector:Conn_Coaxial
Connections:
- net VREF is gone; now on net VCC: C4.1
- net AUDIO: now also J7.1 (In)
- net GND: now also J7.2 (Ext)
- no-connect marks 4 -> 3

Commit message: v3 last board  last version
Parts:
- removed J7: AUDIO, Connector_BarrelJack:BarrelJack_CUI_PJ-063AH_Horizontal_CircularHoles, symbol Connector:Conn_Coaxial
- added J7: Barrel_Jack_MountingPin, Connector_BarrelJack:BarrelJack_CUI_PJ-063AH_Horizontal_CircularHoles, symbol Connector:Barrel_Jack_MountingPin
Connections:
- net AUDIO: now also J7.2
- net GND: now also J7.1, J7.MP (MountPin)
Changed lines of the file:
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@@
+    )
+  )
+  (global_label "GND" (shape input) (at 33.274 78.486 270) (fields_autoplaced)
+    (effects (font (size 1.27 1.27)) (justify right))
+    (property "Intersheetrefs" "${INTERSHEET_REFS}" (at 33.274 85.2623 90)
+      (effects (font (size 1.27 1.27)) (justify right) hide)
     )
   )
@@
     )
   )
-  (global_label "AUDIO" (shape input) (at 31.75 62.23 180) (fields_autoplaced)
-    (effects (font (size 1.27 1.27)) (justify right))
-    (property "Intersheetrefs" "${INTERSHEET_REFS}" (at 23.2198 62.23 0)
-      (effects (font (size 1.27 1.27)) (justify right) hide)
+  (global_label "AUDIO" (shape input) (at 40.894 73.406 0) (fields_autoplaced)
+    (effects (font (size 1.27 1.27)) (justify left))
+    (property "Intersheetrefs" "${INTERSHEET_REFS}" (at 49.4242 73.406 0)
+      (effects (font (size 1.27 1.27)) (justify left) hide)
     )
   )
@@
     )
   )
-  (global_label "GND" (shape input) (at 36.83 67.31 270) (fields_autoplaced)
-    (effects (font (size 1.27 1.27)) (justify right))
-    (property "Intersheetrefs" "${INTERSHEET_REFS}" (at 36.83 74.0863 90)
-      (effects (font (size 1.27 1.27)) (justify right) hide)
+  (global_label "GND" (shape input) (at 40.894 68.326 0) (fields_autoplaced)
+    (effects (font (size 1.27 1.27)) (justify left))
+    (property "Intersheetrefs" "${INTERSHEET_REFS}" (at 47.6703 68.326 0)
+      (effects (font (size 1.27 1.27)) (justify left) hide)
     )
   )
@@
     )
   )
-  (symbol (lib_id "Connector:Conn_Coaxial") (at 36.83 62.23 0) (unit 1)
-    (in_bom yes) (on_board yes) (dnp no) (fields_autoplaced)
-    (property "Reference" "J7" (at 40.005 61.8882 0)
-      (effects (font (size 1.27 1.27)) (justify left))
-    )
-    (property "Value" "AUDIO" (at 40.005 64.4282 0)
-      (effects (font (size 1.27 1.27)) (justify left))
-    )
-    (property "Footprint" "Connector_BarrelJack:BarrelJack_CUI_PJ-063AH_Horizontal_CircularHoles" (at 36.83 62.23 0)
-      (effects (font (size 1.27 1.27)) hide)
-    )
-    (property "Datasheet" " ~" (at 36.83 62.23 0)
-      (effects (font (size 1.27 1.27)) hide)
-    )
-    (pin "1")
-    (pin "2")
-    (instances
-      (project "tn_vdp_v3_board"
-        (path "/e3c6ad0b-efa5-4827-958c-c20bf8519fa1"
-          (reference "J7") (unit 1)
-        )
-      )
-    )
-  )
   (symbol (lib_id "Connector_Generic:Conn_02x10_Odd_Even") (at 74.93 31.75 0) (unit 1)
     (in_bom yes) (on_board yes) (dnp no) (fields_autoplaced)
@@
         )
       )
+    )
+  )
+  (symbol (lib_id "Connector:Barrel_Jack_MountingPin") (at 33.274 70.866 0) (unit 1)
+    (in_bom yes) (on_board yes) (dnp no) (fields_autoplaced)
+    (property "Reference" "J7" (at 33.274 62.992 0)
+      (effects (font (size 1.27 1.27)))
+    )
+    (property "Value" "Barrel_Jack_MountingPin" (at 33.274 65.532 0)
+      (effects (font (size 1.27 1.27)))
+    )
+    (property "Footprint" "Connector_BarrelJack:BarrelJack_CUI_PJ-063AH_Horizontal_CircularHoles" (at 34.544 71.882 0)
+      (effects (font (size 1.27 1.27)) hide)
+    )
+    (property "Datasheet" "~" (at 34.544 71.882 0)
+      (effects (font (size 1.27 1.27)) hide)
+    )
+    (pin "1")
+    (pin "2")
+    (pin "MP")
+    (instances
+      (project "tn_vdp_v3_board"
+        (path "/e3c6ad0b-efa5-4827-958c-c20bf8519fa1"
+          (reference "J7") (unit 1)
+        )
+      )
